File: kicad/pxlboard.kicad_pcb (KiCad board)
At the start: 2 copper layers, 72.8 x 83.8 mm, 80 parts, among them U2 LIS3DHTR

Commit message: feat: add power usb c
Parts:
- removed XIAO RP2040: XIAO-RP2040-SMD, lib:XIAO-RP2040-SMD
- added G***: LOGO, LOGO, B.Cu at (81.9, 56.5)
- added P1: USB_C_Plug_USB2.0, lib:TYPE-C-31-M-12, F.Cu at (79.4, 22.8)
- added U1: XIAO-RP2040-SMD, lib:XIAO-RP2040-SMD, B.Cu at (59.6, 32.0)
- moved C7 9.54 mm to (80.3, 102.2)
- moved C9 9.31 mm to (90.2, 28.8)
Routing:
- net +5V: track 726.5 -> 745.6 mm, vias 1 -> 0
- net unconnected-(P1-SHIELD-PadS1): track 0.00 -> 17.0 mm
- net GND tiny: track 13.8 -> 20.2 mm, vias 2 -> 3
- net GND: track 214.7 -> 220.8 mm, vias 74 -> 73
- net +3.3V: track 30.8 -> 31.3 mm
Other:
- outline, holes or cut-outs redrawn
- board text added: "PxlBoard"
- board text added: "a project by kieran"
